Commit message: fixed end leg joints
 the did not have a axis defined, they (02 12 22 32 42 52) still do not have a correct origin, neither does (00 01)

File: SpiderRobot_pkg/robots/SpiderRobot (copy).URDF (robot description, URDF)
Before this commit: robot SpiderRobot, 19 links, 18 joints
Links:
- link Link_00: geometry collision mesh filename=package://SpiderRobot/meshes/Link_00.STL; visual mesh filename=package://SpiderRobot/meshes/Link_00.STL
- link Link_01: geometry collision mesh filename=package://SpiderRobot/meshes/Link_01.STL; visual mesh filename=package://SpiderRobot/meshes/Link_01.STL
- link Link_02: geometry collision mesh filename=package://SpiderRobot/meshes/Link_02.STL; visual mesh filename=package://SpiderRobot/meshes/Link_02.STL
- link Link_10: geometry collision mesh filename=package://SpiderRobot/meshes/Link_10.STL; visual mesh filename=package://SpiderRobot/meshes/Link_10.STL
- link Link_11: geometry collision mesh filename=package://SpiderRobot/meshes/Link_11.STL; visual mesh filename=package://SpiderRobot/meshes/Link_11.STL
- link Link_12: geometry collision mesh filename=package://SpiderRobot/meshes/Link_12.STL; visual mesh filename=package://SpiderRobot/meshes/Link_12.STL
- link Link_20: geometry collision mesh filename=package://SpiderRobot/meshes/Link_20.STL; visual mesh filename=package://SpiderRobot/meshes/Link_20.STL
- link Link_21: geometry collision mesh filename=package://SpiderRobot/meshes/Link_21.STL; visual mesh filename=package://SpiderRobot/meshes/Link_21.STL
- link Link_22: geometry collision mesh filename=package://SpiderRobot/meshes/Link_22.STL; visual mesh filename=package://SpiderRobot/meshes/Link_22.STL
- link Link_30: geometry collision mesh filename=package://SpiderRobot/meshes/Link_30.STL; visual mesh filename=package://SpiderRobot/meshes/Link_30.STL
- link Link_31: geometry collision mesh filename=package://SpiderRobot/meshes/Link_31.STL; visual mesh filename=package://SpiderRobot/meshes/Link_31.STL
- link Link_32: geometry collision mesh filename=package://SpiderRobot/meshes/Link_32.STL; visual mesh filename=package://SpiderRobot/meshes/Link_32.STL
- link Link_40: geometry collision mesh filename=package://SpiderRobot/meshes/Link_40.STL; visual mesh filename=package://SpiderRobot/meshes/Link_40.STL
- link Link_41: geometry collision mesh filename=package://SpiderRobot/meshes/Link_41.STL; visual mesh filename=package://SpiderRobot/meshes/Link_41.STL
- link Link_42: geometry collision mesh filename=package://SpiderRobot/meshes/Link_42.STL; visual mesh filename=package://SpiderRobot/meshes/Link_42.STL
- link Link_50: geometry collision mesh filename=package://SpiderRobot/meshes/Link_50.STL; visual mesh filename=package://SpiderRobot/meshes/Link_50.STL
- link Link_51: geometry collision mesh filename=package://SpiderRobot/meshes/Link_51.STL; visual mesh filename=package://SpiderRobot/meshes/Link_51.STL
- link Link_52: geometry collision mesh filename=package://SpiderRobot/meshes/Link_52.STL; visual mesh filename=package://SpiderRobot/meshes/Link_52.STL
- link Link_Base: geometry collision mesh filename=package://SpiderRobot/meshes/Link_Base.STL; visual mesh filename=package://SpiderRobot/meshes/Link_Base.STL
Joints:
- joint Joint_00: axis 0 1 0 -> -1 0 0
- joint Joint_02: axis 1 0 0 -> 0 0 0
- joint Joint_10: axis 0 1 0 -> 0 -1 0
- joint Joint_12: axis 1 0 0 -> 0 0 0
- joint Joint_20: axis 0 1 0 -> 0 -1 0
- joint Joint_21: axis -1 0 0 -> 1 0 0
- joint Joint_22: axis 1 0 0 -> 0 0 0
- joint Joint_30: axis 0 1 0 -> 0 -1 0
- joint Joint_31: axis 1 0 0 -> -1 0 0
- joint Joint_32: axis 1 0 0 -> 0 0 0
- joint Joint_40: axis 0 1 0 -> 0 -1 0
- joint Joint_41: axis 1 0 0 -> -1 0 0
- joint Joint_42: axis 1 0 0 -> 0 0 0
- joint Joint_50: axis 0 1 0 -> 0 -1 0
- joint Joint_52: axis 1 0 0 -> 0 0 0
