Commit message: changed extemly low numbers to zero (3.3x10^-15)

File: SpiderRobot_pkg/robots/SpiderRobot.URDF (robot description, URDF)
Before this commit: robot SpiderRobot, 19 links, 18 joints
Joints:
- joint Joint_00: origin xyz=0.21137 -0.09086 0.16867 rpy=-1.5708 -5.3027E-17 -1.0472 -> xyz=0.21137 -0.09086 0.16867 rpy=-1.5708 0 -1.0472
- joint Joint_01: origin xyz=0.08812 -0.02286 0.04445 rpy=1.5708 6.6613E-16 3.1416 -> xyz=0.08812 -0.02286 0.04445 rpy=1.5708 0 3.1416
- joint Joint_20: origin xyz=-0.025655 -0.16469 0.13016 rpy=1.5708 -5.3027E-17 -2.0944 -> xyz=-0.025655 -0.16469 0.13016 rpy=1.5708 0 -2.0944
- joint Joint_21: origin xyz=0 0.038506 0.03683 rpy=3.1416 3.3307E-16 3.1416 -> xyz=0 0.038506 0.03683 rpy=3.1416 0 3.1416
- joint Joint_30: origin xyz=-0.025655 -0.3016 0.13016 rpy=1.5708 -5.3027E-17 -1.0472 -> xyz=-0.025655 -0.3016 0.13016 rpy=1.5708 0 -1.0472
- joint Joint_31: origin xyz=0 0.038506 0.03683 rpy=-3.1416 6.6613E-16 3.4694E-16 -> xyz=0 0.038506 0.03683 rpy=-3.1416 0 0
- joint Joint_32: origin xyz=-0.02413 -0.02286 -0.04445 rpy=-1.5708 -2.498E-15 3.4694E-16 -> xyz=-0.02413 -0.02286 -0.04445 rpy=-1.5708 0 0
- joint Joint_50: origin xyz=0.21147 -0.3016 0.13016 rpy=1.5708 5.3027E-17 1.0472 -> xyz=0.21147 -0.3016 0.13016 rpy=1.5708 0 1.0472
- joint Joint_52: origin xyz=-0.02413 0.02286 0.04445 rpy=1.5708 -2.387E-15 0 -> xyz=-0.02413 0.02286 0.04445 rpy=1.5708 0 0
